File: hardware/board/board.sch (KiCad schematic (older format))
At the start: 51 parts, among them J1 Eurorack Power, J2 USB_MICRO_RIGHT, J3 GATE_IN, J4 GATE_OUT, J5 CV_IN, J6 AUDIO_OUT, J7 Tag-Connect SWD, J8 Big button, Q1 MMBT3904, SW1 TACT_4.2MM, U1 ATSAMD21G18A-AUT, U2 LM7805, U3 AP2112K-3.3, U4 LM4040LP-10, U5 TL072, U6 MCP6001-OT, U7 74AHCT1G125, U8 GD25Q16C

Commit message: Fix incorrect resistor values
Parts:
- R5: value 6.8k -> 100k; mpn ERA-8AEB682V -> (none)
- R6: value 6.8k -> 200k; mpn ERA-8AEB682V -> (none)
- R7: value 6.8k -> 33k; mpn ERA-8AEB682V -> (none)
- renumbered J8 to Button1, J5 to CV_IN1, J3 to GATE_IN1, J4 to GATE_OUT1, J6 to HONK_OUT1, SW1 to RESET1, J7 to SWD1, J2 to USB1
Other:
- note added: "Vin = -5 to +5\nVout = 3.30 to 0.00"
- note removed: "Vin = -5 to +5\nVout = 3.3 to 0"
- moved on the sheet: C16
Changed lines of the file:
@@
 Sheet 1 1
 Title "Big Honking Button"
-Date "2020-03-02"
-Rev "v1"
+Date "2020-03-05"
+Rev "v2"
 Comp "Winterbloom"
 Comment1 "Alethea Flowers"
@@
 P 6150 3600
 F 0 "R5" V 5943 3600 50  0000 C CNN
-F 1 "6.8k" V 6034 3600 50  0000 C CNN
+F 1 "100k" V 6034 3600 50  0000 C CNN
 F 2 "Resistor_SMD:R_1206_3216Metric_Pad1.42x1.75mm_HandSolder" V 6080 3600 50  0001 C CNN
 F 3 "~" H 6150 3600 50  0001 C CNN
-F 4 "ERA-8AEB682V" H 6150 3600 50  0001 C CNN "mpn"
+F 4 "" H 6150 3600 50  0001 C CNN "mpn"
 	1    6150 3600
 	0    1    1    0
@@
 P 6850 4100
 F 0 "R7" V 7050 4100 50  0000 C CNN
-F 1 "6.8k" V 6950 4100 50  0000 C CNN
+F 1 "33k" V 6950 4100 50  0000 C CNN
 F 2 "Resistor_SMD:R_1206_3216Metric_Pad1.42x1.75mm_HandSolder" V 6780 4100 50  0001 C CNN
 F 3 "~" H 6850 4100 50  0001 C CNN
-F 4 "ERA-8AEB682V" H 6850 4100 50  0001 C CNN "mpn"
+F 4 "" H 6850 4100 50  0001 C CNN "mpn"
 	1    6850 4100
 	0    1    1    0
@@
 P 6150 3950
 F 0 "R6" V 5943 3950 50  0000 C CNN
-F 1 "6.8k" V 6034 3950 50  0000 C CNN
+F 1 "200k" V 6034 3950 50  0000 C CNN
 F 2 "Resistor_SMD:R_1206_3216Metric_Pad1.42x1.75mm_HandSolder" V 6080 3950 50  0001 C CNN
 F 3 "~" H 6150 3950 50  0001 C CNN
-F 4 "ERA-8AEB682V" H 6150 3950 50  0001 C CNN "mpn"
+F 4 "" H 6150 3950 50  0001 C CNN "mpn"
 	1    6150 3950
 	0    1    1    0
@@
 $EndComp
 Text Notes 7200 3800 0    50   ~ 0
-Vin = -5 to +5\nVout = 3.3 to 0
+Vin = -5 to +5\nVout = 3.30 to 0.00
 $Comp
 L Device:R R1
@@
 $EndComp
 $Comp
-L Connector:AudioJack2_SwitchT J3
+L Connector:AudioJack2_SwitchT GATE_IN1
 U 1 1 5E572BB3
 P 10500 4450
-F 0 "J3" H 10320 4383 50  0000 R CNN
+F 0 "GATE_IN1" H 10320 4383 50  0000 R CNN
 F 1 "GATE_IN" H 10320 4474 50  0000 R CNN
 F 2 "board:WQP-PJ301M-12_JACK" H 10500 4450 50  0001 C CNN
@@
 $EndComp
 $Comp
-L Connector:AudioJack2_SwitchT J4
+L Connector:AudioJack2_SwitchT GATE_OUT1
 U 1 1 5E574915
 P 10500 5000
-F 0 "J4" H 10320 4933 50  0000 R CNN
+F 0 "GATE_OUT1" H 10320 4933 50  0000 R CNN
 F 1 "GATE_OUT" H 10320 5024 50  0000 R CNN
 F 2 "board:WQP-PJ301M-12_JACK" H 10500 5000 50  0001 C CNN
@@
 $EndComp
 $Comp
-L Connector:AudioJack2_SwitchT J5
+L Connector:AudioJack2_SwitchT CV_IN1
 U 1 1 5E574F97
 P 10500 5550
-F 0 "J5" H 10320 5483 50  0000 R CNN
+F 0 "CV_IN1" H 10320 5483 50  0000 R CNN
 F 1 "CV_IN" H 10320 5574 50  0000 R CNN
 F 2 "board:WQP-PJ301M-12_JACK" H 10500 5550 50  0001 C CNN
@@
 $EndComp
 $Comp
-L Connector:AudioJack2_SwitchT J6
+L Connector:AudioJack2_SwitchT HONK_OUT1
 U 1 1 5E575F38
 P 10500 6050
-F 0 "J6" H 10320 5983 50  0000 R CNN
+F 0 "HONK_OUT1" H 10320 5983 50  0000 R CNN
 F 1 "AUDIO_OUT" H 10320 6074 50  0000 R CNN
 F 2 "board:WQP-PJ301M-12_JACK" H 10500 6050 50  0001 C CNN
@@
 	0    1    1    0
 $EndComp
-$Comp
-L power:+3.3V #PWR0145
-U 1 1 5E59905F
-P 8000 3350
-F 0 "#PWR0145" H 8000 3200 50  0001 C CNN
-F 1 "+3.3V" H 8015 3523 50  0000 C CNN
-F 2 "" H 8000 3350 50  0001 C CNN
-F 3 "" H 8000 3350 50  0001 C CNN
-	1    8000 3350
-	1    0    0    -1
-$EndComp
-$Comp
-L Device:C C16
-U 1 1 5E599CFE
-P 8000 3500
-F 0 "C16" H 8115 3546 50  0000 L CNN
-F 1 "0.1uF" H 8115 3455 50  0000 L CNN
-F 2 "Capacitor_SMD:C_0603_1608Metric_Pad1.05x0.95mm_HandSolder" H 8038 3350 50  0001 C CNN
-F 3 "~" H 8000 3500 50  0001 C CNN
-F 4 "MF-CAP-0603-0.1uF" H 8000 3500 50  0001 C CNN "mpn"
-	1    8000 3500
-	1    0    0    -1
-$EndComp
-$Comp
-L power:GND #PWR0146
-U 1 1 5E59A246
-P 8000 3650
-F 0 "#PWR0146" H 8000 3400 50  0001 C CNN
-F 1 "GND" H 8005 3477 50  0000 C CNN
-F 2 "" H 8000 3650 50  0001 C CNN
-F 3 "" H 8000 3650 50  0001 C CNN
-	1    8000 3650
-	1    0    0    -1
-$EndComp
 Wire Wire Line
 	5350 1500 5500 1500
@@
 Connection ~ 5350 1500
 $Comp
-L MF_Connectors:USB_MICRO_RIGHT J2
+L MF_Connectors:USB_MICRO_RIGHT USB1
 U 1 1 5E6974D5
 P 9050 4900
-F 0 "J2" H 8822 4892 45  0000 R CNN
+F 0 "USB1" H 8822 4892 45  0000 R CNN
 F 1 "USB_MICRO_RIGHT" H 8822 4808 45  0000 R CNN
 F 2 "MF_Connectors:MF_Connectors-MICROUSB-RIGHT" V 8818 4754 20  0001 C CNN
@@
 $EndComp
 $Comp
-L MF_Switches:TACT_4.2MM SW1
+L MF_Switches:TACT_4.2MM RESET1
 U 1 1 5E69D81E
 P 3600 7500
-F 0 "SW1" H 3600 7770 45  0000 C CNN
+F 0 "RESET1" H 3600 7770 45  0000 C CNN
 F 1 "TACT_4.2MM" H 3600 7686 45  0000 C CNN
 F 2 "MF_Switches:MF_Switches-TACT4.2MM" H 3490 7650 20  0001 L CNN
@@
 NoConn ~ 6400 7150
 $Comp
-L Connector_Generic:Conn_02x03_Counter_Clockwise J7
+L Connector_Generic:Conn_02x03_Counter_Clockwise SWD1
 U 1 1 5E668F1F
 P 6100 7250
-F 0 "J7" H 6150 7567 50  0000 C CNN
+F 0 "SWD1" H 6150 7567 50  0000 C CNN
 F 1 "Tag-Connect SWD" H 6150 7476 50  0000 C CNN
 F 2 "Connector:Tag-Connect_TC2030-IDC-NL_2x03_P1.27mm_Vertical" H 6100 7250 50  0001 C CNN
@@
 $EndComp
 $Comp
-L Connector_Generic:Conn_01x02 J8
+L Connector_Generic:Conn_01x02 Button1
 U 1 1 5E75A93E
 P 9100 6000
-F 0 "J8" H 9180 5992 50  0000 L CNN
+F 0 "Button1" H 9180 5992 50  0000 L CNN
 F 1 "Big button" H 9180 5901 50  0000 L CNN
 F 2 "Connector_PinHeader_2.54mm:PinHeader_1x02_P2.54mm_Vertical" H 9100 6000 50  0001 C CNN
@@
 Text GLabel 8900 6000 0    50   Input ~ 0
 D9
+$Comp
+L power:GND #PWR0146
+U 1 1 5E59A246
+P 8200 3600
+F 0 "#PWR0146" H 8200 3350 50  0001 C CNN
+F 1 "GND" H 8205 3427 50  0000 C CNN
+F 2 "" H 8200 3600 50  0001 C CNN
+F 3 "" H 8200 3600 50  0001 C CNN
+	1    8200 3600
+	1    0    0    -1
+$EndComp
+$Comp
+L Device:C C16
+U 1 1 5E599CFE
+P 8200 3450
+F 0 "C16" H 8315 3496 50  0000 L CNN
+F 1 "0.1uF" H 8315 3405 50  0000 L CNN
+F 2 "Capacitor_SMD:C_0603_1608Metric_Pad1.05x0.95mm_HandSolder" H 8238 3300 50  0001 C CNN
+F 3 "~" H 8200 3450 50  0001 C CNN
+F 4 "MF-CAP-0603-0.1uF" H 8200 3450 50  0001 C CNN "mpn"
+	1    8200 3450
+	1    0    0    -1
+$EndComp
+$Comp
+L power:+3.3V #PWR0145
+U 1 1 5E59905F
+P 8200 3300
+F 0 "#PWR0145" H 8200 3150 50  0001 C CNN
+F 1 "+3.3V" H 8215 3473 50  0000 C CNN
+F 2 "" H 8200 3300 50  0001 C CNN
+F 3 "" H 8200 3300 50  0001 C CNN
+	1    8200 3300
+	1    0    0    -1
+$EndComp
 $EndSCHEMATC

Commit message: Fix issues found in the first prototype
Parts:
- D1, D2: mpn 1N4148W-7-F -> MF-DIO-SOD123-1N4148
- J1: mpn CONN-08671 -> 61201021621
- Q1: symbol Transistor_BJT:2N3904 -> Transistor_BJT:MMBT3904; mpn MMBT3904 -> MF-DSC-SOT233-MMBT3904
- R5: mpn (none) -> ERA-8AEB104V
- R6: value 200k -> 510k; mpn (none) -> ERA-8AEB514V
- R7: value 33k -> 82k; mpn (none) -> ERA-8AEB823V
- U6: mpn MCP6001RT-I/OT -> MCP6001T-I/OT
Other:
- note added: "Vin = -2 to +2\nVout = 3.22 to 0.03"
- note removed: "Vin = -5 to +5\nVout = 3.30 to 0.00"
Changed lines of the file:
@@
 Sheet 1 1
 Title "Big Honking Button"
-Date "2020-03-05"
-Rev "v2"
+Date "2020-03-19"
+Rev "v3"
 Comp "Winterbloom"
 Comment1 "Alethea Flowers"
@@
 $EndComp
 $Comp
-L Transistor_BJT:2N3904 Q1
+L Transistor_BJT:MMBT3904 Q1
 U 1 1 5E4A636D
 P 10250 1450
@@
 F 2 "Package_TO_SOT_SMD:SOT-23" H 10450 1375 50  0001 L CIN
 F 3 "https://www.fairchildsemi.com/datasheets/2N/2N3904.pdf" H 10250 1450 50  0001 L CNN
-F 4 "MMBT3904" H 10250 1450 50  0001 C CNN "mpn"
+F 4 "MF-DSC-SOT233-MMBT3904" H 10250 1450 50  0001 C CNN "mpn"
 	1    10250 1450
 	1    0    0    -1
@@
 F 2 "Package_TO_SOT_SMD:SOT-23-5" H 6750 3300 50  0001 L CNN
 F 3 "http://ww1.microchip.com/downloads/en/DeviceDoc/21733j.pdf" H 6850 3700 50  0001 C CNN
-F 4 "MCP6001RT-I/OT" H 6850 3500 50  0001 C CNN "mpn"
+F 4 "MCP6001T-I/OT" H 6850 3500 50  0001 C CNN "mpn"
 	1    6850 3500
 	1    0    0    -1
@@
 F 2 "Resistor_SMD:R_1206_3216Metric_Pad1.42x1.75mm_HandSolder" V 6080 3600 50  0001 C CNN
 F 3 "~" H 6150 3600 50  0001 C CNN
-F 4 "" H 6150 3600 50  0001 C CNN "mpn"
+F 4 "ERA-8AEB104V" H 6150 3600 50  0001 C CNN "mpn"
 	1    6150 3600
 	0    1    1    0
@@
 P 6850 4100
 F 0 "R7" V 7050 4100 50  0000 C CNN
-F 1 "33k" V 6950 4100 50  0000 C CNN
+F 1 "82k" V 6950 4100 50  0000 C CNN
 F 2 "Resistor_SMD:R_1206_3216Metric_Pad1.42x1.75mm_HandSolder" V 6780 4100 50  0001 C CNN
 F 3 "~" H 6850 4100 50  0001 C CNN
-F 4 "" H 6850 4100 50  0001 C CNN "mpn"
+F 4 "ERA-8AEB823V" H 6850 4100 50  0001 C CNN "mpn"
 	1    6850 4100
 	0    1    1    0
@@
 P 6150 3950
 F 0 "R6" V 5943 3950 50  0000 C CNN
-F 1 "200k" V 6034 3950 50  0000 C CNN
+F 1 "510k" V 6034 3950 50  0000 C CNN
 F 2 "Resistor_SMD:R_1206_3216Metric_Pad1.42x1.75mm_HandSolder" V 6080 3950 50  0001 C CNN
 F 3 "~" H 6150 3950 50  0001 C CNN
-F 4 "" H 6150 3950 50  0001 C CNN "mpn"
+F 4 "ERA-8AEB514V" H 6150 3950 50  0001 C CNN "mpn"
 	1    6150 3950
 	0    1    1    0
@@
 $EndComp
 Text Notes 7200 3800 0    50   ~ 0
-Vin = -5 to +5\nVout = 3.30 to 0.00
+Vin = -2 to +2\nVout = 3.22 to 0.03
 $Comp
 L Device:R R1
@@
 F 2 "SF Connectors:2X5-SHROUDED_LOCK" H 1050 1550 20  0001 C CNN
 F 3 "" H 1050 1150 50  0001 C CNN
-F 4 "CONN-08671" H 1050 1150 50  0001 C CNN "mpn"
+F 4 "61201021621" H 1050 1150 50  0001 C CNN "mpn"
 	1    1050 1150
 	1    0    0    -1
@@
 F 2 "Diode_SMD:D_SOD-123" H 1450 1350 50  0001 C CNN
 F 3 "~" H 1450 1350 50  0001 C CNN
-F 4 "1N4148W-7-F" H 1450 1350 50  0001 C CNN "mpn"
+F 4 "MF-DIO-SOD123-1N4148" H 1450 1350 50  0001 C CNN "mpn"
 	1    1450 1350
 	-1   0    0    1
@@
 F 2 "Diode_SMD:D_SOD-123" H 1450 950 50  0001 C CNN
 F 3 "~" H 1450 950 50  0001 C CNN
-F 4 "1N4148W-7-F" H 1450 950 50  0001 C CNN "mpn"
+F 4 "MF-DIO-SOD123-1N4148" H 1450 950 50  0001 C CNN "mpn"
 	1    1450 950
 	1    0    0    -1
@@
 U 1 1 5E6DE131
 P 4050 4950
-F 0 "R12" H 3900 5000 50  0000 L CNN
+F 0 "R12" H 3850 5000 50  0000 L CNN
 F 1 "10k" H 3850 4900 50  0000 L CNN
 F 2 "Resistor_SMD:R_1206_3216Metric_Pad1.42x1.75mm_HandSolder" V 3980 4950 50  0001 C CNN

Commit message: Fix pinout on zener diode
Parts:
- removed U4: LM4040LP-10, Package_TO_SOT_SMD:SOT-23, symbol Reference_Voltage:LM4040LP-10
- added U4: LM4040DBZ-10, Package_TO_SOT_SMD:SOT-23, symbol Reference_Voltage:LM4040DBZ-10
- R10, R11: footprint Resistor_SMD:R_1206_3216Metric_Pad1.42x1.75mm_HandSolder -> Resistor_SMD:R_0805_2012Metric_Pad1.15x1.40mm_HandSolder; mpn ERA-8AEB102V -> MF-RES-0805-1K
- R12, R9: footprint Resistor_SMD:R_1206_3216Metric_Pad1.42x1.75mm_HandSolder -> Resistor_SMD:R_0805_2012Metric_Pad1.15x1.40mm_HandSolder; mpn ERA-8AEB103V -> MF-RES-0805-10K
Changed lines of the file:
@@
 Sheet 1 1
 Title "Big Honking Button"
-Date "2020-03-19"
-Rev "v3"
+Date "2020-04-15"
+Rev "v4"
 Comp "Winterbloom"
 Comment1 "Alethea Flowers"
@@
 F 0 "R9" H 10280 1054 50  0000 R CNN
 F 1 "10k" H 10280 1145 50  0000 R CNN
-F 2 "Resistor_SMD:R_1206_3216Metric_Pad1.42x1.75mm_HandSolder" V 10280 1100 50  0001 C CNN
+F 2 "Resistor_SMD:R_0805_2012Metric_Pad1.15x1.40mm_HandSolder" V 10280 1100 50  0001 C CNN
 F 3 "~" H 10350 1100 50  0001 C CNN
-F 4 "ERA-8AEB103V" H 10350 1100 50  0001 C CNN "mpn"
+F 4 "MF-RES-0805-10K" H 10350 1100 50  0001 C CNN "mpn"
 	1    10350 1100
 	-1   0    0    1
@@
 	1    6750 3200
 	1    0    0    -1
-$EndComp
-$Comp
-L Reference_Voltage:LM4040LP-10 U4
-U 1 1 5E4BA161
-P 4200 3350
-F 0 "U4" V 4150 3150 50  0000 L CNN
-F 1 "LM4040LP-10" V 4250 2700 50  0000 L CNN
-F 2 "Package_TO_SOT_SMD:SOT-23" H 4200 3150 50  0001 C CIN
-F 3 "http://www.ti.com/lit/ds/symlink/lm4040-n.pdf" H 4200 3350 50  0001 C CIN
-F 4 "LM4040DIM3-10.0/NOPB" H 4200 3350 50  0001 C CNN "mpn"
-	1    4200 3350
-	0    1    1    0
 $EndComp
 Text Notes 7200 3800 0    50   ~ 0
@@
 Text GLabel 4650 3200 2    50   Input ~ 0
 VREF_-10
-Connection ~ 4200 3200
 $Comp
 L Device:C C10
@@
 Wire Wire Line
 	4400 3500 4200 3500
-Connection ~ 4200 3500
 Wire Wire Line
 	4400 3200 4650 3200
@@
 F 0 "R11" V 8393 1250 50  0000 C CNN
 F 1 "1k" V 8484 1250 50  0000 C CNN
-F 2 "Resistor_SMD:R_1206_3216Metric_Pad1.42x1.75mm_HandSolder" V 8530 1250 50  0001 C CNN
+F 2 "Resistor_SMD:R_0805_2012Metric_Pad1.15x1.40mm_HandSolder" V 8530 1250 50  0001 C CNN
 F 3 "~" H 8600 1250 50  0001 C CNN
-F 4 "ERA-8AEB102V" H 8600 1250 50  0001 C CNN "mpn"
+F 4 "MF-RES-0805-1K" H 8600 1250 50  0001 C CNN "mpn"
 	1    8600 1250
 	0    1    1    0
@@
 F 0 "R10" V 5893 1150 50  0000 C CNN
 F 1 "1k" V 5984 1150 50  0000 C CNN
-F 2 "Resistor_SMD:R_1206_3216Metric_Pad1.42x1.75mm_HandSolder" V 6030 1150 50  0001 C CNN
+F 2 "Resistor_SMD:R_0805_2012Metric_Pad1.15x1.40mm_HandSolder" V 6030 1150 50  0001 C CNN
 F 3 "~" H 6100 1150 50  0001 C CNN
-F 4 "ERA-8AEB102V" H 6100 1150 50  0001 C CNN "mpn"
+F 4 "MF-RES-0805-1K" H 6100 1150 50  0001 C CNN "mpn"
 	1    6100 1150
 	0    1    1    0
@@
 F 0 "R12" H 3850 5000 50  0000 L CNN
 F 1 "10k" H 3850 4900 50  0000 L CNN
-F 2 "Resistor_SMD:R_1206_3216Metric_Pad1.42x1.75mm_HandSolder" V 3980 4950 50  0001 C CNN
+F 2 "Resistor_SMD:R_0805_2012Metric_Pad1.15x1.40mm_HandSolder" V 3980 4950 50  0001 C CNN
 F 3 "~" H 4050 4950 50  0001 C CNN
-F 4 "ERA-8AEB103V" H 4050 4950 50  0001 C CNN "mpn"
+F 4 "MF-RES-0805-10K" H 4050 4950 50  0001 C CNN "mpn"
 	1    4050 4950
 	1    0    0    -1
@@
 	1    0    0    -1
 $EndComp
+$Comp
+L Reference_Voltage:LM4040DBZ-10 U4
+U 1 1 5E97DED0
+P 4200 3350
+F 0 "U4" V 4250 3100 50  0000 L CNN
+F 1 "LM4040DBZ-10" V 4150 2650 50  0000 L CNN
+F 2 "Package_TO_SOT_SMD:SOT-23" H 4200 3150 50  0001 C CIN
+F 3 "http://www.ti.com/lit/ds/symlink/lm4040-n.pdf" H 4200 3350 50  0001 C CIN
+F 4 "LM4040DIM3-10.0/NOPB" H 4200 3350 50  0001 C CNN "mpn"
+	1    4200 3350
+	0    1    1    0
+$EndComp
+Connection ~ 4200 3200
+Connection ~ 4200 3500
 $EndSCHEMATC

Commit message: Update board
Parts:
- R1, R10, R11, R12, R13, R2, R3, R4, R5, R6, R7, R8, R9: symbol Device:R -> Device:R_US
Changed lines of the file:
@@
 EESchema Schematic File Version 4
-LIBS:board-cache
-EELAYER 29 0
+EELAYER 30 0
 EELAYER END
 $Descr A4 11693 8268
@@
 $EndComp
 $Comp
-L Device:R R2
+L Device:R_US R2
 U 1 1 5E48CFC1
 P 4800 1400
@@
 $EndComp
 $Comp
-L Device:R R4
+L Device:R_US R4
 U 1 1 5E490A91
 P 5650 1500
@@
 Connection ~ 4800 1250
 $Comp
-L Device:R R3
+L Device:R_US R3
 U 1 1 5E48FF0C
 P 4950 1250
@@
 $EndComp
 $Comp
-L Device:R R8
+L Device:R_US R8
 U 1 1 5E4A526F
 P 9900 1450
@@
 $EndComp
 $Comp
-L Device:R R9
+L Device:R_US R9
 U 1 1 5E4A57F0
 P 10350 1100
@@
 $EndComp
 $Comp
-L Device:R R5
+L Device:R_US R5
 U 1 1 5E4B2A88
 P 6150 3600
@@
 $EndComp
 $Comp
-L Device:R R7
+L Device:R_US R7
 U 1 1 5E4B2F81
 P 6850 4100
@@
 Connection ~ 6550 3600
 $Comp
-L Device:R R6
+L Device:R_US R6
 U 1 1 5E4B5FFD
 P 6150 3950
@@
 Vin = -2 to +2\nVout = 3.22 to 0.03
 $Comp
-L Device:R R1
+L Device:R_US R1
 U 1 1 5E4BC7EA
 P 4200 3050
@@
 Connection ~ 7150 4100
 $Comp
-L Device:R R11
+L Device:R_US R11
 U 1 1 5E5547AE
 P 8600 1250
@@
 $EndComp
 $Comp
-L Device:R R10
+L Device:R_US R10
 U 1 1 5E555614
 P 6100 1150
@@
 	1    0    0    -1
 $EndComp
-$Comp
-L power:GND #PWR0148
-U 1 1 5E69FB3A
-P 3500 7600
-F 0 "#PWR0148" H 3500 7350 50  0001 C CNN
-F 1 "GND" H 3505 7427 50  0000 C CNN
-F 2 "" H 3500 7600 50  0001 C CNN
-F 3 "" H 3500 7600 50  0001 C CNN
-	1    3500 7600
-	0    1    1    0
-$EndComp
 Text GLabel 1000 6900 0    50   Input ~ 0
 RESET
@@
 	4000 5100 4050 5100
 $Comp
-L Device:R R12
+L Device:R_US R12
 U 1 1 5E6DE131
 P 4050 4950
@@
 $EndComp
 $Comp
-L Device:R R13
+L Device:R_US R13
 U 1 1 5E6E6D2E
 P 4650 6400
@@
 Connection ~ 4200 3200
 Connection ~ 4200 3500
+$Comp
+L power:GND #PWR0148
+U 1 1 5E69FB3A
+P 3500 7600
+F 0 "#PWR0148" H 3500 7350 50  0001 C CNN
+F 1 "GND" H 3505 7427 50  0000 C CNN
+F 2 "" H 3500 7600 50  0001 C CNN
+F 3 "" H 3500 7600 50  0001 C CNN
+	1    3500 7600
+	0    1    1    0
+$EndComp
 $EndSCHEMATC
