File: hardware/board/board.sch (KiCad schematic (older format))
At the start: 51 parts, among them J1 Eurorack Power, Q1 MMBT3904, U1 ATSAMD21G18A-AUT, U2 LM7805, U3 AP2112K-3.3, U4 LM4040DBZ-10, U5 TL072, U6 MCP6001-OT, U7 74AHCT1G125, U8 GD25Q16C

Commit message: Board revision v5
- Switch to 8mb flash
- Switch all resistors to 0603
- Change CV input to -5 to +5
Parts:
- J1: symbol SparkFun-Connectors:CONN_05X2SHD_LOCK -> board-rescue:CONN_05X2SHD_LOCK-SparkFun-Connectors
- R1: footprint Resistor_SMD:R_1206_3216Metric_Pad1.42x1.75mm_HandSolder -> Resistor_SMD:R_0603_1608Metric_Pad1.05x0.95mm_HandSolder; mpn ERA-8AEB222V -> ERA-3AED222V
- R10, R11: footprint Resistor_SMD:R_0805_2012Metric_Pad1.15x1.40mm_HandSolder -> Resistor_SMD:R_0603_1608Metric_Pad1.05x0.95mm_HandSolder; mpn MF-RES-0805-1K -> MF-RES-0603-1K
- R12, R9: footprint Resistor_SMD:R_0805_2012Metric_Pad1.15x1.40mm_HandSolder -> Resistor_SMD:R_0603_1608Metric_Pad1.05x0.95mm_HandSolder; mpn MF-RES-0805-10K -> MF-RES-0603-10K
- R13: value 2.2k -> 1k; footprint Resistor_SMD:R_1206_3216Metric_Pad1.42x1.75mm_HandSolder -> Resistor_SMD:R_0603_1608Metric_Pad1.05x0.95mm_HandSolder; mpn ERA-8AEB222V -> MF-RES-0603-1K
- R2, R4: footprint Resistor_SMD:R_1206_3216Metric_Pad1.42x1.75mm_HandSolder -> Resistor_SMD:R_0603_1608Metric_Pad1.05x0.95mm_HandSolder; mpn ERA-8AEB473V -> ERA-3AED473V
- R3: footprint Resistor_SMD:R_1206_3216Metric_Pad1.42x1.75mm_HandSolder -> Resistor_SMD:R_0603_1608Metric_Pad1.05x0.95mm_HandSolder; mpn ERA-8AEB682V -> ERA-3AED682V
- R5, R8: footprint Resistor_SMD:R_1206_3216Metric_Pad1.42x1.75mm_HandSolder -> Resistor_SMD:R_0603_1608Metric_Pad1.05x0.95mm_HandSolder; mpn ERA-8AEB104V -> ERA-3AED104V
- R6: value 510k -> 200k; footprint Resistor_SMD:R_1206_3216Metric_Pad1.42x1.75mm_HandSolder -> Resistor_SMD:R_0603_1608Metric_Pad1.05x0.95mm_HandSolder; mpn ERA-8AEB514V -> ERA-3AEB204V
- R7: value 82k -> 33k; footprint Resistor_SMD:R_1206_3216Metric_Pad1.42x1.75mm_HandSolder -> Resistor_SMD:R_0603_1608Metric_Pad1.05x0.95mm_HandSolder; mpn ERA-8AEB823V -> ERA-3AED333V
- RESET1: symbol MF_Switches:TACT_4.2MM -> board-rescue:TACT_4.2MM-MF_Switches
- U8: value GD25Q16C -> GD25Q64C; symbol board:GD25Q16C -> board:GD25Q64C; mfn GD25Q16CSIGR -> GD25Q64CSIGR; mpn GD25Q16CSIGR -> GD25Q64CSIGR
- USB1: symbol MF_Connectors:USB_MICRO_RIGHT -> board-rescue:USB_MICRO_RIGHT-MF_Connectors
Connections:
- net GND: now also U1.19 (PB10)
- no-connect marks 13 -> 12
Other:
- note added: "Grounded for v5+"
- note added: "Vin = -5 to +5\nVout = 3.3 to 0.00"
- note removed: "Vin = -2 to +2\nVout = 3.22 to 0.03"
Changed lines of the file:
@@
 Sheet 1 1
 Title "Big Honking Button"
-Date "2020-04-15"
-Rev "v4"
+Date "2020-10-07"
+Rev "v5"
 Comp "Winterbloom"
 Comment1 "Alethea Flowers"
@@
 Text GLabel 3000 3800 2    50   Input ~ 0
 A5
-NoConn ~ 3000 4200
 NoConn ~ 3000 4300
 Text GLabel 4500 1250 0    50   Input ~ 0
@@
 F 0 "R2" H 4730 1354 50  0000 R CNN
 F 1 "47k" H 4730 1445 50  0000 R CNN
-F 2 "Resistor_SMD:R_1206_3216Metric_Pad1.42x1.75mm_HandSolder" V 4730 1400 50  0001 C CNN
+F 2 "Resistor_SMD:R_0603_1608Metric_Pad1.05x0.95mm_HandSolder" V 4730 1400 50  0001 C CNN
 F 3 "~" H 4800 1400 50  0001 C CNN
-F 4 "ERA-8AEB473V" H 4800 1400 50  0001 C CNN "mpn"
+F 4 "ERA-3AED473V" H 4800 1400 50  0001 C CNN "mpn"
 	1    4800 1400
 	-1   0    0    1
@@
 F 0 "R4" V 5850 1500 50  0000 C CNN
 F 1 "47k" V 5750 1500 50  0000 C CNN
-F 2 "Resistor_SMD:R_1206_3216Metric_Pad1.42x1.75mm_HandSolder" V 5580 1500 50  0001 C CNN
+F 2 "Resistor_SMD:R_0603_1608Metric_Pad1.05x0.95mm_HandSolder" V 5580 1500 50  0001 C CNN
 F 3 "~" H 5650 1500 50  0001 C CNN
-F 4 "ERA-8AEB473V" H 5650 1500 50  0001 C CNN "mpn"
+F 4 "ERA-3AED473V" H 5650 1500 50  0001 C CNN "mpn"
 	1    5650 1500
 	0    -1   1    0
@@
 F 0 "R3" V 4743 1250 50  0000 C CNN
 F 1 "6.8k" V 4834 1250 50  0000 C CNN
-F 2 "Resistor_SMD:R_1206_3216Metric_Pad1.42x1.75mm_HandSolder" V 4880 1250 50  0001 C CNN
+F 2 "Resistor_SMD:R_0603_1608Metric_Pad1.05x0.95mm_HandSolder" V 4880 1250 50  0001 C CNN
 F 3 "~" H 4950 1250 50  0001 C CNN
-F 4 "ERA-8AEB682V" H 4950 1250 50  0001 C CNN "mpn"
+F 4 "ERA-3AED682V" H 4950 1250 50  0001 C CNN "mpn"
 	1    4950 1250
 	0    1    1    0
@@
 F 0 "R8" V 9693 1450 50  0000 C CNN
 F 1 "100k" V 9784 1450 50  0000 C CNN
-F 2 "Resistor_SMD:R_1206_3216Metric_Pad1.42x1.75mm_HandSolder" V 9830 1450 50  0001 C CNN
+F 2 "Resistor_SMD:R_0603_1608Metric_Pad1.05x0.95mm_HandSolder" V 9830 1450 50  0001 C CNN
 F 3 "~" H 9900 1450 50  0001 C CNN
-F 4 "ERA-8AEB104V" H 9900 1450 50  0001 C CNN "mpn"
+F 4 "ERA-3AED104V" H 9900 1450 50  0001 C CNN "mpn"
 	1    9900 1450
 	0    1    1    0
@@
 F 0 "R9" H 10280 1054 50  0000 R CNN
 F 1 "10k" H 10280 1145 50  0000 R CNN
-F 2 "Resistor_SMD:R_0805_2012Metric_Pad1.15x1.40mm_HandSolder" V 10280 1100 50  0001 C CNN
+F 2 "Resistor_SMD:R_0603_1608Metric_Pad1.05x0.95mm_HandSolder" V 10280 1100 50  0001 C CNN
 F 3 "~" H 10350 1100 50  0001 C CNN
-F 4 "MF-RES-0805-10K" H 10350 1100 50  0001 C CNN "mpn"
+F 4 "MF-RES-0603-10K" H 10350 1100 50  0001 C CNN "mpn"
 	1    10350 1100
 	-1   0    0    1
@@
 F 0 "R5" V 5943 3600 50  0000 C CNN
 F 1 "100k" V 6034 3600 50  0000 C CNN
-F 2 "Resistor_SMD:R_1206_3216Metric_Pad1.42x1.75mm_HandSolder" V 6080 3600 50  0001 C CNN
+F 2 "Resistor_SMD:R_0603_1608Metric_Pad1.05x0.95mm_HandSolder" V 6080 3600 50  0001 C CNN
 F 3 "~" H 6150 3600 50  0001 C CNN
-F 4 "ERA-8AEB104V" H 6150 3600 50  0001 C CNN "mpn"
+F 4 "ERA-3AED104V" H 6150 3600 50  0001 C CNN "mpn"
 	1    6150 3600
 	0    1    1    0
@@
 P 6850 4100
 F 0 "R7" V 7050 4100 50  0000 C CNN
-F 1 "82k" V 6950 4100 50  0000 C CNN
-F 2 "Resistor_SMD:R_1206_3216Metric_Pad1.42x1.75mm_HandSolder" V 6780 4100 50  0001 C CNN
+F 1 "33k" V 6950 4100 50  0000 C CNN
+F 2 "Resistor_SMD:R_0603_1608Metric_Pad1.05x0.95mm_HandSolder" V 6780 4100 50  0001 C CNN
 F 3 "~" H 6850 4100 50  0001 C CNN
-F 4 "ERA-8AEB823V" H 6850 4100 50  0001 C CNN "mpn"
+F 4 "ERA-3AED333V" H 6850 4100 50  0001 C CNN "mpn"
 	1    6850 4100
 	0    1    1    0
@@
 P 6150 3950
 F 0 "R6" V 5943 3950 50  0000 C CNN
-F 1 "510k" V 6034 3950 50  0000 C CNN
-F 2 "Resistor_SMD:R_1206_3216Metric_Pad1.42x1.75mm_HandSolder" V 6080 3950 50  0001 C CNN
+F 1 "200k" V 6034 3950 50  0000 C CNN
+F 2 "Resistor_SMD:R_0603_1608Metric_Pad1.05x0.95mm_HandSolder" V 6080 3950 50  0001 C CNN
 F 3 "~" H 6150 3950 50  0001 C CNN
-F 4 "ERA-8AEB514V" H 6150 3950 50  0001 C CNN "mpn"
+F 4 "ERA-3AEB204V" H 6150 3950 50  0001 C CNN "mpn"
 	1    6150 3950
 	0    1    1    0
@@
 $EndComp
 Text Notes 7200 3800 0    50   ~ 0
-Vin = -2 to +2\nVout = 3.22 to 0.03
+Vin = -5 to +5\nVout = 3.3 to 0.00
 $Comp
 L Device:R_US R1
@@
 F 0 "R1" H 4130 3004 50  0000 R CNN
 F 1 "2.2k" H 4130 3095 50  0000 R CNN
-F 2 "Resistor_SMD:R_1206_3216Metric_Pad1.42x1.75mm_HandSolder" V 4130 3050 50  0001 C CNN
+F 2 "Resistor_SMD:R_0603_1608Metric_Pad1.05x0.95mm_HandSolder" V 4130 3050 50  0001 C CNN
 F 3 "~" H 4200 3050 50  0001 C CNN
-F 4 "ERA-8AEB222V" H 4200 3050 50  0001 C CNN "mpn"
+F 4 "ERA-3AED222V" H 4200 3050 50  0001 C CNN "mpn"
 	1    4200 3050
 	-1   0    0    1
@@
 Connection ~ 4400 3200
 $Comp
-L SparkFun-Connectors:CONN_05X2SHD_LOCK J1
+L board-rescue:CONN_05X2SHD_LOCK-SparkFun-Connectors J1
 U 1 1 5E4C5788
 P 1050 1150
@@
 F 0 "R11" V 8393 1250 50  0000 C CNN
 F 1 "1k" V 8484 1250 50  0000 C CNN
-F 2 "Resistor_SMD:R_0805_2012Metric_Pad1.15x1.40mm_HandSolder" V 8530 1250 50  0001 C CNN
+F 2 "Resistor_SMD:R_0603_1608Metric_Pad1.05x0.95mm_HandSolder" V 8530 1250 50  0001 C CNN
 F 3 "~" H 8600 1250 50  0001 C CNN
-F 4 "MF-RES-0805-1K" H 8600 1250 50  0001 C CNN "mpn"
+F 4 "MF-RES-0603-1K" H 8600 1250 50  0001 C CNN "mpn"
 	1    8600 1250
 	0    1    1    0
@@
 F 0 "R10" V 5893 1150 50  0000 C CNN
 F 1 "1k" V 5984 1150 50  0000 C CNN
-F 2 "Resistor_SMD:R_0805_2012Metric_Pad1.15x1.40mm_HandSolder" V 6030 1150 50  0001 C CNN
+F 2 "Resistor_SMD:R_0603_1608Metric_Pad1.05x0.95mm_HandSolder" V 6030 1150 50  0001 C CNN
 F 3 "~" H 6100 1150 50  0001 C CNN
-F 4 "MF-RES-0805-1K" H 6100 1150 50  0001 C CNN "mpn"
+F 4 "MF-RES-0603-1K" H 6100 1150 50  0001 C CNN "mpn"
 	1    6100 1150
 	0    1    1    0
@@
 Connection ~ 5350 1500
 $Comp
-L MF_Connectors:USB_MICRO_RIGHT USB1
+L board-rescue:USB_MICRO_RIGHT-MF_Connectors USB1
 U 1 1 5E6974D5
 P 9050 4900
@@
 $EndComp
 $Comp
-L MF_Switches:TACT_4.2MM RESET1
+L board-rescue:TACT_4.2MM-MF_Switches RESET1
 U 1 1 5E69D81E
 P 3600 7500
@@
 unused
 $Comp
-L board:GD25Q16C U8
+L board:GD25Q64C U8
 U 1 1 5E6D95D1
 P 4650 5200
 F 0 "U8" H 4800 5650 50  0000 C CNN
-F 1 "GD25Q16C" H 4950 5550 50  0000 C CNN
+F 1 "GD25Q64C" H 4950 5550 50  0000 C CNN
 F 2 "Package_SO:SOIC-8_5.23x5.23mm_P1.27mm" H 4650 5200 50  0001 C CNN
 F 3 "http://www.winbond.com/resource-files/w25q32jv%20revg%2003272018%20plus.pdf" H 4650 5200 50  0001 C CNN
-F 4 "GD25Q16CSIGR" H 4650 5200 50  0001 C CNN "mfn"
-F 5 "GD25Q16CSIGR" H 4650 5200 50  0001 C CNN "mpn"
+F 4 "GD25Q64CSIGR" H 4650 5200 50  0001 C CNN "mfn"
+F 5 "GD25Q64CSIGR" H 4650 5200 50  0001 C CNN "mpn"
 	1    4650 5200
 	1    0    0    -1
@@
 F 0 "R12" H 3850 5000 50  0000 L CNN
 F 1 "10k" H 3850 4900 50  0000 L CNN
-F 2 "Resistor_SMD:R_0805_2012Metric_Pad1.15x1.40mm_HandSolder" V 3980 4950 50  0001 C CNN
+F 2 "Resistor_SMD:R_0603_1608Metric_Pad1.05x0.95mm_HandSolder" V 3980 4950 50  0001 C CNN
 F 3 "~" H 4050 4950 50  0001 C CNN
-F 4 "MF-RES-0805-10K" H 4050 4950 50  0001 C CNN "mpn"
+F 4 "MF-RES-0603-10K" H 4050 4950 50  0001 C CNN "mpn"
 	1    4050 4950
 	1    0    0    -1
@@
 P 4650 6400
 F 0 "R13" H 4580 6354 50  0000 R CNN
-F 1 "2.2k" H 4580 6445 50  0000 R CNN
-F 2 "Resistor_SMD:R_1206_3216Metric_Pad1.42x1.75mm_HandSolder" V 4580 6400 50  0001 C CNN
+F 1 "1k" H 4580 6445 50  0000 R CNN
+F 2 "Resistor_SMD:R_0603_1608Metric_Pad1.05x0.95mm_HandSolder" V 4580 6400 50  0001 C CNN
 F 3 "~" H 4650 6400 50  0001 C CNN
-F 4 "ERA-8AEB222V" H 4650 6400 50  0001 C CNN "mpn"
+F 4 "MF-RES-0603-1K" H 4650 6400 50  0001 C CNN "mpn"
 	1    4650 6400
 	-1   0    0    1
@@
 	0    1    1    0
 $EndComp
+Wire Wire Line
+	3000 4200 3850 4200
+$Comp
+L power:GND #PWR0161
+U 1 1 5F90F093
+P 3850 4200
+F 0 "#PWR0161" H 3850 3950 50  0001 C CNN
+F 1 "GND" H 3855 4027 50  0000 C CNN
+F 2 "" H 3850 4200 50  0001 C CNN
+F 3 "" H 3850 4200 50  0001 C CNN
+	1    3850 4200
+	1    0    0    -1
+$EndComp
+Text Notes 3550 4200 0    50   ~ 0
+Grounded for v5+
 $EndSCHEMATC

Commit message: Add PDF of the schematic and a pre-submit hook to make sure it doesn't go out of sync.
Parts:
- Button1: mpn (none) -> OBSF-30
Changed lines of the file:
@@
 F 2 "Connector_PinHeader_2.54mm:PinHeader_1x02_P2.54mm_Vertical" H 9100 6000 50  0001 C CNN
 F 3 "~" H 9100 6000 50  0001 C CNN
+F 4 "OBSF-30" H 9100 6000 50  0001 C CNN "mpn"
 	1    9100 6000
 	1    0    0    -1
