File: hardware/board/board.kicad_pcb (KiCad board)
At the start: 2 copper layers, 40.1 x 49.3 mm, 54 parts, among them J1 Eurorack Power, Q1 MMBT3904, U1 ATSAMD21G18A-AUT, U2 LM7805, U3 AP2112K-3.3, U4 LM4040DBZ-10, U5 TL072, U6 MCP6001-OT, U7 74AHCT1G125, U8 GD25Q64C

Commit message: Switch to KiCAD 6
Other:
- net class Default removed
