File: hardware/board/analog-outs.kicad_sch (KiCad schematic)
At the start: 24 parts, among them U6 TL072

Commit message: hardware: rename to Goosehonk Nebula, prep v7
Other:
- note added: "Gain = 3.3 Low-pass corner frequency = ~800kHz"
- note added: "PWM DAC: - PWM Freq: - 8 bit = 186 kHz - 9 bit = 93 kHz - 10 bit = 46 kHz - 11 bit = 23 kHz (Verified) - 12 bit = 11 kHz (Verified) - Filter topology: 3rd order multiple feeback (MFB) low-pass - Calculator: http://sim.okawa-denshi.jp/en/Multiple3tool.php - Gain: -3.125 - Fc1 = ~5 kHz, Fc2 = ~3 kHz - Q = ~0.6, ζ = ~0.8 - Falstad: https://tinyurl.com/2cdxc5kc"
- note removed: "Gain = Low-pass corner frequency ="
- note removed: "PWM DAC: - PWM Freq: - 8 bit = 186 kHz - 9 bit = 93 kHz - 10 bit = 46 kHz - 11 bit = 23 kHz - 12 bit = 11 kHz - Filter topology: 3rd order multiple feeback (MFB) low-pass - Calculator: http://sim.okawa-denshi.jp/en/Multiple3tool.php - Gain: -3.125 - Fc1 = ~5 kHz, Fc2 = ~3 kHz - Q = ~0.6, ζ = ~0.8 - Falstad: https://tinyurl.com/2cdxc5kc"
- title: Big Honking Button -> Goosehonk Nebula
- moved on the sheet: C?, J?, R?, TP?, U6A, U6B, U6C
