File: hardware/board/board.kicad_sch (KiCad schematic)
At the start: 0 parts

Commit message: hardware: rename to Goosehonk Nebula, prep v7
Other:
- note removed: "TODO: - Make sure both analog outputs can deal with clock output"
- title: Big Honking Button -> Goosehonk Nebula
