File: hardware/board/power.kicad_sch (KiCad schematic)
At the start: 20 parts

Commit message: hardware: rename to Goosehonk Nebula, prep v7
Other:
- title: Big Honking Button -> Goosehonk Nebula
Changed lines of the file:
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@@
   (paper "USLetter")
   (title_block
-    (title "Big Honking Button")
-    (date "2023-08-02")
-    (rev "v5")
+    (title "Goosehonk Nebula")
+    (date "2023-10-08")
+    (rev "v7")
     (company "Winterbloom")
     (comment 1 "Alethea Flowers")
     (comment 2 "CERN-OHL-P V2")
+    (comment 3 "goose.wntr.dev")
   )
   (junction (at 113.03 38.1) (diameter 0) (color 0 0 0 0)
